Commit message: config: measured hardware calibration, OpenCR udev rules, arm torque relax
- Firmware: confirmed XM430 IDs/limits for lm_arm and wheel_clock, RELAX/HOLD
  keywords (torque off/on in place), gripper current scale.
- Control: measured arm joint offsets/directions, LM meters-per-rad mapping,
  gripper grasp squeeze angle, keep arm/LM/gripper targets across new tasks.
- URDF and meshes resized to measured link lengths; fit_measured.py helper.
- config/udev: OpenCR rules keyed by USB path (arm/LM 2.1, wheel/clock 2.2.2
  after the 2026-10-26 hardware change) and LiDAR rules for the Jetson.
- craft_dashboard.sh launch groups, motor axis jog bench test.

Co-Authored-By: Claude Opus 5.5 <noreply@anthropic.com>

File: src/craft_planning/v75_ws/src/v75_arm_ik/urdf/v75_robot.urdf (robot description, URDF)
Before this commit: robot v75_robot, 28 links, 27 joints
Joints:
- joint elbow_joint: limit lower=-1.52541776624 upper=2.83790536374 effort=0 velocity=0 -> lower=-1.4379 upper=3.3618 effort=0 velocity=0; origin xyz=1.11022302463e-16 0.0764664888983 0.171746546037 rpy=0 0 0 -> xyz=0 0.077280 0.173574 rpy=0 0 0
- joint idler_joint: origin xyz=0.234 0.0563662 0.0955 rpy=0 0 0 -> xyz=0.22164 0.0563662 0.0955 rpy=0 0 0
- joint jaw_lower_joint: mimic (none) -> joint=jaw_upper_joint multiplier=1 offset=0
- joint shoulder_joint: limit lower=-1.15191730632 upper=1.98967534727 effort=0 velocity=0 -> lower=-0.3848 upper=2.0237 effort=0 velocity=0
- joint slide_joint: axis 1 0 0 -> -1 0 0; limit lower=-0.072 upper=0.032 effort=0 velocity=0 -> lower=-0.0320 upper=0.0630 effort=0 velocity=0; origin xyz=0.02 0 0 rpy=0 0 0 -> xyz=-0.00135 0 0 rpy=0 0 0
- joint tool_roll_joint: limit lower=-1.74532925199 upper=1.74532925199 effort=0 velocity=0 -> lower=-4.7226 upper=3.8295 effort=0 velocity=0; origin xyz=2.77555756156e-17 0.056 1.11022302463e-16 rpy=0 0 0 -> xyz=0 0.055 0 rpy=0 0 0
- joint tool_tcp_joint: origin xyz=0 0.1024 0 rpy=0 0 0 -> xyz=0 0.1101 0 rpy=0 0 0
- joint wrist_pitch_joint: limit lower=-1.67900674042 upper=1.98618468877 effort=0 velocity=0 -> lower=-0.4370 upper=1.5876 effort=0 velocity=0; origin xyz=2.77555756156e-16 0.0835666144223 0.0451842998617 rpy=0 0 0 -> xyz=0 0.089498 0.021309 rpy=0 0 0

Commit message: arm: measured geometry, 0.5 deg tolerances, least-elbow-load IK, board tooling
- URDF (both copies): shoulder axis 114 mm above the floor (was 122.25), elbow 187 mm,
  elbow->wrist 95 mm, wrist->tool-roll horn 78 mm, TCP 0.118 (mid usable grip), slide and
  wrist/tool-roll limits from measured motor ranges; meshes refit (fit_measured.py).
- ArmPlanner: collect every distinct IK solution (seed + fixed-seed restarts) and return the
  one with the least elbow gravity moment, nearest the seed on ties; new branch test, FK
  expectation updated for TCP 0.118 and the 114 mm shoulder.
- Arm and LM arrival tolerance 0.5 motor deg in firmware lm_arm and control.yaml (kept equal);
  position I gain on the arm joints, single-turn axis unwrap at boot.
- udev: arm/LM is the OpenCR on 2.2.2, any other OpenCR is wheel/clock; ModemManager ignored.
- firmware/usb_to_dxl: ROBOTIS passthrough sketch for DYNAMIXEL Wizard (wizard helper);
  test/motor_axis_jog removed in favour of Wizard.
- Docs: IK branch choice, tolerance match, Wizard board lock.

Co-Authored-By: Claude Opus 5.5 <noreply@anthropic.com>

File: src/craft_planning/v75_ws/src/v75_arm_ik/urdf/v75_robot.urdf (robot description, URDF)
Before this commit: robot v75_robot, 28 links, 27 joints
Joints:
- joint elbow_joint: origin xyz=0 0.077280 0.173574 rpy=0 0 0 -> xyz=0 0.076060 0.170833 rpy=0 0 0
- joint shoulder_joint: origin xyz=0.129 0.051 0.12225 rpy=0 0 0 -> xyz=0.129 0.051 0.114 rpy=0 0 0
- joint slide_joint: limit lower=-0.0320 upper=0.0630 effort=0 velocity=0 -> lower=-0.0438 upper=0.0630 effort=0 velocity=0
- joint tool_roll_joint: limit lower=-4.7226 upper=3.8295 effort=0 velocity=0 -> lower=-4.6250 upper=1.4835 effort=0 velocity=0; origin xyz=0 0.055 0 rpy=0 0 0 -> xyz=0 0.078 0 rpy=0 0 0
- joint tool_tcp_joint: origin xyz=0 0.1101 0 rpy=0 0 0 -> xyz=0 0.118 0 rpy=0 0 0
- joint wrist_pitch_joint: limit lower=-0.4370 upper=1.5876 effort=0 velocity=0 -> lower=-2.1822 upper=2.3537 effort=0 velocity=0; origin xyz=0 0.089498 0.021309 rpy=0 0 0 -> xyz=0 0.092417 0.022004 rpy=0 0 0
