Commit message: lying scenario testing

File: src/craft_planning/v75_ws/src/v75_arm_ik/urdf/v75_robot.urdf (robot description, URDF)
Before this commit: robot v75_robot, 28 links, 27 joints
Joints:
- joint elbow_joint: limit lower=-1.4379 upper=3.3618 effort=0 velocity=0 -> lower=-1.4379 upper=3.4490 effort=0 velocity=0
- joint wrist_pitch_joint: limit lower=-2.1822 upper=2.3537 effort=0 velocity=0 -> lower=-2.3655 upper=2.3537 effort=0 velocity=0
